File: Arduino_MEGA_2560-Rev3.sch (EAGLE design)
At the start: 38 parts

Commit message: Version 0.1 - Faltan planos de tierra
Parts:
- added R17, R18, R22, R23, R24, R26, R27, R28, R29: (no value), rcl:R-US_0207/15
Connections:
- removed net N$10: ADCH.3, R7.2
- removed net N$21: ADCH.4, R8.2
- removed net N$22: ADCH.5, U$3.CTS
- removed net N$23: ADCH.6, U$3.DTR
- removed net N$24: ADCH.7, U$3.RTS
- removed net N$25: ADCH.8, U$3.RX
- new net N$29: R17.1, U$6.3.3V, U$6.GND
- new net N$32: R22.1, U$6.TX
- new net N$33: R18.1, U$6.RST
- new net N$34: R24.1, U$5.3.3V, U$5.GND
- new net N$35: R23.1, U$4.3.3V, U$4.GND
- new net N$40: R28.1, U$5.TX
- new net N$41: R29.1, U$5.RST
- new net N$42: R26.2, U$4.TX
- new net N$43: R27.1, U$4.RST
- net GND: now also R17.2, R23.2, R24.2; no longer U$4.3.3V, U$4.GND, U$5.3.3V, U$5.GND, U$6.3.3V, U$6.GND
- net PA0: now also R7.2
- net PA1: now also R8.2
- net PA2: now also U$3.RTS
- net PA3: now also U$3.RX
- net PA4: now also U$3.CTS
- net PA5: now also U$3.DTR
- net PA6: now also R26.1
- net PA7: now also R27.2
- net PC0: now also U$6.RX
- net PC1: now also U$6.RTS
- net PC2: now also R18.2
- net PC3: now also R22.2
- net PC4: now also U$4.DTR
- net PC5: now also U$4.CTS
- net PC6: now also U$4.RX
- net PC7: now also U$4.RTS
- net PD7: now also U$6.CTS
- net PE3: now also U$5.RX
- net PE4: now also U$5.CTS
- net PE5: now also U$5.DTR
- net PG2: now also U$6.DTR
- net PG5: now also U$5.RTS
- net PH3: now also R28.2
- net PH4: now also R29.2
Other:
- moved on the sheet: R7, R8, U$4, U$5, U$6

Commit message: Terminada la version 1.0
Parts:
- added COMMUNICATION1: 8x1F-H8.5, SmartPrj:PINHD-1X8
- added JP1: (no value), pinhead:PINHD-1X6
Connections:
- new net N$10: ADCH.3, JP1.1
- new net N$21: ADCH.4, JP1.2
- new net N$22: ADCH.5, JP1.3
- new net N$23: ADCH.6, JP1.4
- new net N$24: ADCH.7, JP1.5
- new net N$25: ADCH.8, JP1.6
- net RXD1: now also COMMUNICATION1.3
- net RXD2: now also COMMUNICATION1.5
- net RXD3: now also COMMUNICATION1.7
- net SCL: now also COMMUNICATION1.1
- net SDA: now also COMMUNICATION1.2
- net TXD1: now also COMMUNICATION1.4
- net TXD2: now also COMMUNICATION1.6
- net TXD3: now also COMMUNICATION1.8
Changed lines of the file:
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@@
 <part name="R28" library="rcl" deviceset="R-US_" device="0207/15"/>
 <part name="R29" library="rcl" deviceset="R-US_" device="0207/15"/>
+<part name="JP1" library="pinhead" deviceset="PINHD-1X6" device=""/>
+<part name="COMMUNICATION1" library="SmartPrj" deviceset="PINHD-1X8" device="" value="8x1F-H8.5"/>
 </parts>
 <sheets>
@@
 </instance>
 <instance part="COMMUNICATION" gate="A" x="482.6" y="48.26" smashed="yes" rot="MR180">
-<attribute name="NAME" x="492.125" y="48.26" size="1.778" layer="95" rot="MR180"/>
+<attribute name="NAME" x="433.705" y="53.34" size="1.778" layer="95" rot="MR180"/>
 <attribute name="VALUE" x="476.25" y="60.96" size="1.778" layer="96" rot="MR180"/>
 </instance>
@@
 <attribute name="NAME" x="422.91" y="16.2814" size="1.778" layer="95" rot="R180"/>
 <attribute name="VALUE" x="422.91" y="18.542" size="1.778" layer="96" rot="R180"/>
+</instance>
+<instance part="JP1" gate="A" x="91.44" y="40.64"/>
+<instance part="COMMUNICATION1" gate="A" x="497.84" y="48.26" smashed="yes" rot="MR180">
+<attribute name="NAME" x="507.365" y="35.56" size="1.778" layer="95" rot="MR180"/>
+<attribute name="VALUE" x="491.49" y="60.96" size="1.778" layer="96" rot="MR180"/>
 </instance>
 </instances>
@@
 <label x="428.625" y="41.275" size="1.778" layer="95"/>
 <pinref part="COMMUNICATION" gate="A" pin="2"/>
+<pinref part="COMMUNICATION1" gate="A" pin="2"/>
+<wire x1="495.3" y1="40.64" x2="480.06" y2="40.64" width="0.1524" layer="91"/>
+<junction x="480.06" y="40.64"/>
 </segment>
 </net>
@@
 <label x="428.625" y="38.735" size="1.778" layer="95"/>
 <pinref part="COMMUNICATION" gate="A" pin="1"/>
+<pinref part="COMMUNICATION1" gate="A" pin="1"/>
+<wire x1="495.3" y1="38.1" x2="480.06" y2="38.1" width="0.1524" layer="91"/>
+<junction x="480.06" y="38.1"/>
 </segment>
 </net>
@@
 <label x="464.185" y="43.815" size="1.778" layer="95"/>
 <pinref part="COMMUNICATION" gate="A" pin="3"/>
+<pinref part="COMMUNICATION1" gate="A" pin="3"/>
+<wire x1="495.3" y1="43.18" x2="480.06" y2="43.18" width="0.1524" layer="91"/>
+<junction x="480.06" y="43.18"/>
 </segment>
 </net>
@@
 <label x="464.185" y="46.355" size="1.778" layer="95"/>
 <pinref part="COMMUNICATION" gate="A" pin="4"/>
+<pinref part="COMMUNICATION1" gate="A" pin="4"/>
+<wire x1="495.3" y1="45.72" x2="480.06" y2="45.72" width="0.1524" layer="91"/>
+<junction x="480.06" y="45.72"/>
 </segment>
 </net>
@@
 <label x="464.185" y="48.895" size="1.778" layer="95"/>
 <pinref part="COMMUNICATION" gate="A" pin="5"/>
+<pinref part="COMMUNICATION1" gate="A" pin="5"/>
+<wire x1="495.3" y1="48.26" x2="480.06" y2="48.26" width="0.1524" layer="91"/>
+<junction x="480.06" y="48.26"/>
 </segment>
 </net>
@@
 <label x="464.185" y="53.975" size="1.778" layer="95"/>
 <pinref part="COMMUNICATION" gate="A" pin="7"/>
+<pinref part="COMMUNICATION1" gate="A" pin="7"/>
+<wire x1="495.3" y1="53.34" x2="480.06" y2="53.34" width="0.1524" layer="91"/>
+<junction x="480.06" y="53.34"/>
 </segment>
 </net>
@@
 <label x="464.185" y="51.435" size="1.778" layer="95"/>
 <pinref part="COMMUNICATION" gate="A" pin="6"/>
+<pinref part="COMMUNICATION1" gate="A" pin="6"/>
+<wire x1="495.3" y1="50.8" x2="480.06" y2="50.8" width="0.1524" layer="91"/>
+<junction x="480.06" y="50.8"/>
 </segment>
 </net>
@@
 <label x="464.185" y="56.515" size="1.778" layer="95"/>
 <pinref part="COMMUNICATION" gate="A" pin="8"/>
+<pinref part="COMMUNICATION1" gate="A" pin="8"/>
+<wire x1="495.3" y1="55.88" x2="480.06" y2="55.88" width="0.1524" layer="91"/>
+<junction x="480.06" y="55.88"/>
 </segment>
 </net>
@@
 </segment>
 </net>
+<net name="N$10" class="0">
+<segment>
+<pinref part="ADCH" gate="A" pin="3"/>
+<wire x1="71.12" y1="50.8" x2="83.82" y2="50.8" width="0.1524" layer="91"/>
+<wire x1="83.82" y1="50.8" x2="83.82" y2="48.26" width="0.1524" layer="91"/>
+<pinref part="JP1" gate="A" pin="1"/>
+<wire x1="83.82" y1="48.26" x2="88.9" y2="48.26" width="0.1524" layer="91"/>
+</segment>
+</net>
+<net name="N$21" class="0">
+<segment>
+<pinref part="ADCH" gate="A" pin="4"/>
+<wire x1="71.12" y1="48.26" x2="81.28" y2="48.26" width="0.1524" layer="91"/>
+<wire x1="81.28" y1="48.26" x2="81.28" y2="45.72" width="0.1524" layer="91"/>
+<pinref part="JP1" gate="A" pin="2"/>
+<wire x1="81.28" y1="45.72" x2="88.9" y2="45.72" width="0.1524" layer="91"/>
+</segment>
+</net>
+<net name="N$22" class="0">
+<segment>
+<pinref part="ADCH" gate="A" pin="5"/>
+<wire x1="71.12" y1="45.72" x2="78.74" y2="45.72" width="0.1524" layer="91"/>
+<wire x1="78.74" y1="45.72" x2="78.74" y2="43.18" width="0.1524" layer="91"/>
+<pinref part="JP1" gate="A" pin="3"/>
+<wire x1="78.74" y1="43.18" x2="88.9" y2="43.18" width="0.1524" layer="91"/>
+</segment>
+</net>
+<net name="N$23" class="0">
+<segment>
+<pinref part="ADCH" gate="A" pin="6"/>
+<wire x1="71.12" y1="43.18" x2="76.2" y2="43.18" width="0.1524" layer="91"/>
+<wire x1="76.2" y1="43.18" x2="76.2" y2="40.64" width="0.1524" layer="91"/>
+<pinref part="JP1" gate="A" pin="4"/>
+<wire x1="76.2" y1="40.64" x2="88.9" y2="40.64" width="0.1524" layer="91"/>
+</segment>
+</net>
+<net name="N$24" class="0">
+<segment>
+<pinref part="ADCH" gate="A" pin="7"/>
+<wire x1="71.12" y1="40.64" x2="73.66" y2="40.64" width="0.1524" layer="91"/>
+<wire x1="73.66" y1="40.64" x2="73.66" y2="38.1" width="0.1524" layer="91"/>
+<pinref part="JP1" gate="A" pin="5"/>
+<wire x1="73.66" y1="38.1" x2="88.9" y2="38.1" width="0.1524" layer="91"/>
+</segment>
+</net>
+<net name="N$25" class="0">
+<segment>
+<pinref part="ADCH" gate="A" pin="8"/>
+<wire x1="71.12" y1="38.1" x2="71.12" y2="35.56" width="0.1524" layer="91"/>
+<pinref part="JP1" gate="A" pin="6"/>
+<wire x1="71.12" y1="35.56" x2="88.9" y2="35.56" width="0.1524" layer="91"/>
+</segment>
+</net>

Commit message: Terminada la version 1.0
Connections:
- net GND renamed COUT_GND
- net +5V: no longer R2.2
- net N$25: now also R2.2
Other:
- moved on the sheet: LED1, LED2, R1, R2
Changed lines of the file:
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@@
 <attribute name="VALUE" x="45.72" y="-25.4" size="1.778" layer="96" rot="R90"/>
 </instance>
-<instance part="P+5" gate="1" x="2.54" y="187.96" smashed="yes">
-<attribute name="VALUE" x="4.445" y="190.5" size="1.778" layer="96" rot="R180"/>
+<instance part="P+5" gate="1" x="63.5" y="22.86" smashed="yes">
+<attribute name="VALUE" x="65.405" y="25.4" size="1.778" layer="96" rot="R180"/>
 </instance>
 <instance part="ADCL" gate="A" x="66.04" y="93.98" smashed="yes" rot="MR0">
@@
 <attribute name="VALUE" x="353.06" y="187.96" size="1.778" layer="96" rot="R180"/>
 </instance>
-<instance part="LED1" gate="G$1" x="2.54" y="165.1" smashed="yes">
-<attribute name="NAME" x="6.096" y="160.528" size="1.778" layer="95" rot="R90"/>
-<attribute name="VALUE" x="8.255" y="160.528" size="1.778" layer="96" rot="R90"/>
-</instance>
-<instance part="LED2" gate="G$1" x="15.24" y="165.1" smashed="yes">
-<attribute name="NAME" x="18.796" y="160.528" size="1.778" layer="95" rot="R90"/>
-<attribute name="VALUE" x="20.955" y="160.528" size="1.778" layer="96" rot="R90"/>
-</instance>
-<instance part="R1" gate="G$1" x="2.54" y="175.26" smashed="yes" rot="R90">
-<attribute name="NAME" x="1.0414" y="171.45" size="1.778" layer="95" rot="R90"/>
-<attribute name="VALUE" x="5.842" y="171.45" size="1.778" layer="96" rot="R90"/>
-</instance>
-<instance part="GND3" gate="1" x="2.54" y="149.86" smashed="yes">
-<attribute name="VALUE" x="0" y="147.32" size="1.778" layer="96"/>
-</instance>
-<instance part="R2" gate="G$1" x="15.24" y="175.26" smashed="yes" rot="R90">
-<attribute name="NAME" x="13.7414" y="171.45" size="1.778" layer="95" rot="R90"/>
-<attribute name="VALUE" x="18.542" y="171.45" size="1.778" layer="96" rot="R90"/>
+<instance part="LED1" gate="G$1" x="63.5" y="0" smashed="yes">
+<attribute name="NAME" x="67.056" y="-4.572" size="1.778" layer="95" rot="R90"/>
+<attribute name="VALUE" x="69.215" y="-4.572" size="1.778" layer="96" rot="R90"/>
+</instance>
+<instance part="LED2" gate="G$1" x="76.2" y="0" smashed="yes">
+<attribute name="NAME" x="79.756" y="-4.572" size="1.778" layer="95" rot="R90"/>
+<attribute name="VALUE" x="81.915" y="-4.572" size="1.778" layer="96" rot="R90"/>
+</instance>
+<instance part="R1" gate="G$1" x="63.5" y="10.16" smashed="yes" rot="R90">
+<attribute name="NAME" x="62.0014" y="6.35" size="1.778" layer="95" rot="R90"/>
+<attribute name="VALUE" x="66.802" y="6.35" size="1.778" layer="96" rot="R90"/>
+</instance>
+<instance part="GND3" gate="1" x="63.5" y="-15.24" smashed="yes">
+<attribute name="VALUE" x="60.96" y="-17.78" size="1.778" layer="96"/>
+</instance>
+<instance part="R2" gate="G$1" x="76.2" y="10.16" smashed="yes" rot="R90">
+<attribute name="NAME" x="74.7014" y="6.35" size="1.778" layer="95" rot="R90"/>
+<attribute name="VALUE" x="79.502" y="6.35" size="1.778" layer="96" rot="R90"/>
 </instance>
 <instance part="GND6" gate="1" x="160.02" y="78.74" smashed="yes" rot="R180">
@@
 <pinref part="P+5" gate="1" pin="+5V"/>
 <pinref part="R1" gate="G$1" pin="2"/>
-<wire x1="2.54" y1="185.42" x2="2.54" y2="182.88" width="0.1524" layer="91"/>
-<pinref part="R2" gate="G$1" pin="2"/>
-<wire x1="2.54" y1="182.88" x2="2.54" y2="180.34" width="0.1524" layer="91"/>
-<wire x1="15.24" y1="180.34" x2="15.24" y2="182.88" width="0.1524" layer="91"/>
-<wire x1="15.24" y1="182.88" x2="2.54" y2="182.88" width="0.1524" layer="91"/>
-<junction x="2.54" y="182.88"/>
-</segment>
-</net>
-<net name="GND" class="2">
+<wire x1="63.5" y1="20.32" x2="63.5" y2="15.24" width="0.1524" layer="91"/>
+</segment>
+</net>
+<net name="COUT_GND" class="0">
 <segment>
 <wire x1="480.06" y1="99.06" x2="464.82" y2="99.06" width="0.1524" layer="91"/>
@@
 <pinref part="LED1" gate="G$1" pin="C"/>
 <pinref part="GND3" gate="1" pin="GND"/>
-<wire x1="2.54" y1="160.02" x2="2.54" y2="154.94" width="0.1524" layer="91"/>
+<wire x1="63.5" y1="-5.08" x2="63.5" y2="-10.16" width="0.1524" layer="91"/>
 <pinref part="LED2" gate="G$1" pin="C"/>
-<wire x1="2.54" y1="154.94" x2="2.54" y2="152.4" width="0.1524" layer="91"/>
-<wire x1="15.24" y1="160.02" x2="15.24" y2="154.94" width="0.1524" layer="91"/>
-<wire x1="15.24" y1="154.94" x2="2.54" y2="154.94" width="0.1524" layer="91"/>
-<junction x="2.54" y="154.94"/>
+<wire x1="63.5" y1="-10.16" x2="63.5" y2="-12.7" width="0.1524" layer="91"/>
+<wire x1="76.2" y1="-5.08" x2="76.2" y2="-10.16" width="0.1524" layer="91"/>
+<wire x1="76.2" y1="-10.16" x2="63.5" y2="-10.16" width="0.1524" layer="91"/>
+<junction x="63.5" y="-10.16"/>
 </segment>
 <segment>
@@
 <pinref part="R1" gate="G$1" pin="1"/>
 <pinref part="LED1" gate="G$1" pin="A"/>
-<wire x1="2.54" y1="170.18" x2="2.54" y2="167.64" width="0.1524" layer="91"/>
+<wire x1="63.5" y1="5.08" x2="63.5" y2="2.54" width="0.1524" layer="91"/>
 </segment>
 </net>
@@
 <pinref part="R2" gate="G$1" pin="1"/>
 <pinref part="LED2" gate="G$1" pin="A"/>
-<wire x1="15.24" y1="170.18" x2="15.24" y2="167.64" width="0.1524" layer="91"/>
+<wire x1="76.2" y1="5.08" x2="76.2" y2="2.54" width="0.1524" layer="91"/>
 </segment>
 </net>
@@
 <net name="N$25" class="0">
 <segment>
+<pinref part="R2" gate="G$1" pin="2"/>
+<wire x1="76.2" y1="15.24" x2="76.2" y2="17.78" width="0.1524" layer="91"/>
 <pinref part="ADCH" gate="A" pin="8"/>
 <wire x1="71.12" y1="38.1" x2="71.12" y2="35.56" width="0.1524" layer="91"/>
 <pinref part="JP1" gate="A" pin="6"/>
-<wire x1="71.12" y1="35.56" x2="88.9" y2="35.56" width="0.1524" layer="91"/>
-</segment>
-</net>
+<wire x1="71.12" y1="35.56" x2="81.28" y2="35.56" width="0.1524" layer="91"/>
+<wire x1="81.28" y1="35.56" x2="88.9" y2="35.56" width="0.1524" layer="91"/>
+<wire x1="76.2" y1="17.78" x2="81.28" y2="17.78" width="0.1524" layer="91"/>
+<wire x1="81.28" y1="17.78" x2="81.28" y2="35.56" width="0.1524" layer="91"/>
+<junction x="81.28" y="35.56"/>
+</segment>
+</net>
